File: HalogenDimmer.kicad_pcb (KiCad board)
At the start: 2 copper layers, 19.8 x 63 mm, 31 parts, among them J1 SPI, J5 INPUT_SIGNALS, Q2 IRL2905, Q3 BC817, Q4 BC817, U1 MAX809, U2 ATtiny85-20SU, U3 NCP1117LPST50T3G, U4 MCP1402, Y1 Crystal_GND24

Commit message: HW changes
Other:
- net class Default removed
