File: HalogenDimmer.kicad_sch (KiCad schematic)
At the start: 31 parts, among them J1 SPI, J5 INPUT_SIGNALS, Q2 IRL2905, Q3 BC817, Q4 BC817, U1 MAX809, U2 ATtiny85-20SU, U3 NCP1117LPST50T3G, U4 MCP1402, Y1 Crystal_GND24

Commit message: HW changes
Parts:
- C1, C2: value 22p -> (none); footprint Capacitors_SMD.pretty:C_0805_HandSoldering -> (none)
- C3: value 22m/20V -> (none); footprint Capacitors_Tantalum_SMD:CP_Tantalum_Case-B_EIA-3528-21_Hand -> (none)
- C4, C5, C7: value 100n -> (none); footprint Capacitors_SMD.pretty:C_1206_HandSoldering -> (none)
- C6: value 47m/10V -> (none); footprint Capacitors_Tantalum_SMD:CP_Tantalum_Case-B_EIA-3528-21_Hand -> (none)
- C8: value 1m/10V -> (none); footprint Capacitors_Tantalum_SMD:CP_Tantalum_Case-B_EIA-3528-21_Hand -> (none)
- C9: value 1000m/16v -> (none); footprint Capacitors_ThroughHole:C_Disc_D4.3mm_W1.9mm_P5.00mm -> (none)
- D1, D2: value NP -> (none); footprint Diodes_SMD:D_MicroMELF_Hadsoldering -> (none)
- D3, D5: value 1n4148 -> (none); footprint Diodes_SMD:D_MicroMELF_Hadsoldering -> (none)
- D4: value 5V1 -> (none); footprint Diodes_SMD.pretty:MiniMELF_Handsoldering -> (none)
- J1: value SPI -> (none); footprint Pin_Headers.pretty:Pin_Header_Straight_2x03 -> (none)
- J5: value INPUT_SIGNALS -> (none); footprint Connectors_Molex:Molex_MiniFit-JR-5569-06A2_2x03x4.20mm_Angled -> (none)
- Q2: value IRL2905 -> (none); footprint TO_SOT_Packages_SMD.pretty:TO-252-2Lead -> (none)
- Q3, Q4: value BC817 -> (none); footprint TO_SOT_Packages_SMD.pretty:SOT-23_Handsoldering -> (none)
- R1, R3, R4, R5: value 1k -> (none); footprint Resistors_SMD.pretty:R_0805_HandSoldering -> (none)
- R2, R6, R7: value 10k -> (none); footprint Resistors_SMD.pretty:R_0805_HandSoldering -> (none)
- U1: value MAX809 -> (none); footprint TO_SOT_Packages_SMD.pretty:SOT-23_Handsoldering -> (none)
- U2: value ATtiny85-20SU -> (none); footprint Housings_SOIC:SO-8_5.3x6.2mm_Pitch1.27mm -> (none)
- U3: value NCP1117LPST50T3G -> (none); footprint TO_SOT_Packages_SMD:SOT-223-3_TabPin2 -> (none)
- U4: value MCP1402 -> (none); footprint TO_SOT_Packages_SMD.pretty:SOT-23-5 -> (none)
- Y1: value Crystal_GND24 -> (none); footprint Crystals:Crystal_SMD_3225-4pin_3.2x2.5mm_HandSoldering -> (none)
Connections:
- net GND: no longer C9.2
Other:
- note added: "not needed, attiny85 has internal reset circuit"
- note removed: "not needed, attiny85 has internal reset circute"
